File: udemy-learn-kicad-v6-and-stm32-hardware-design.kicad_sch (KiCad schematic)
At the start: 14 parts, among them SW1 SW_SPDT, U1 STM32F103C8T6, Y1 16MHz

Commit message: PCB layout completed
Parts:
- added C1, C2: 22u, Capacitor_Tantalum_SMD:CP_EIA-3216-18_Kemet-A, symbol Device:C_Polarized
- added C12, C13: 15p, Capacitor_SMD:C_0402_1005Metric, symbol Device:C
- added D1: RED, LED_SMD:LED_0603_1608Metric, symbol Device:LED
- added J1: USB_B_Micro, Connector_USB:USB_Micro-B_Wuerth_629105150521, symbol Connector:USB_B_Micro
- added J2, J3, J4: Conn_01x04_Pin, Connector_PinHeader_2.54mm:PinHeader_1x04_P2.54mm_Vertical, symbol Connector:Conn_01x04_Pin
- added R1: 1k, Resistor_SMD:R_0402_1005Metric, symbol Device:R
- added R3: 1k5, Resistor_SMD:R_0402_1005Metric, symbol Device:R
- added R4, R5: 2k2, Resistor_SMD:R_0402_1005Metric, symbol Device:R
- added U1: AMS1117-3.3, Package_TO_SOT_SMD:SOT-223-3_TabPin2, symbol Regulator_Linear:AMS1117-3.3
- C10: renamed from C8; footprint (none) -> Capacitor_SMD:C_0402_1005Metric
- C11: renamed from C9; footprint (none) -> Capacitor_SMD:C_0402_1005Metric
- C3: renamed from C1; footprint (none) -> Capacitor_SMD:C_0603_1608Metric
- C4: renamed from C2; footprint (none) -> Capacitor_SMD:C_0402_1005Metric
- C5: renamed from C3; footprint (none) -> Capacitor_SMD:C_0402_1005Metric
- C6: renamed from C4; footprint (none) -> Capacitor_SMD:C_0402_1005Metric
- C7: renamed from C5; footprint (none) -> Capacitor_SMD:C_0402_1005Metric
- C8: renamed from C6; value 10n -> 0.1u; footprint (none) -> Capacitor_SMD:C_0402_1005Metric
- C9: renamed from C7; footprint (none) -> Capacitor_SMD:C_0402_1005Metric
- FB1: footprint (none) -> Inductor_SMD:L_0603_1608Metric
- R2: renamed from R1; value 10K -> 10k; footprint (none) -> Resistor_SMD:R_0402_1005Metric
- SW1: footprint (none) -> Button_Switch_THT:SW_E-Switch_EG1224_SPDT_Angled
- Y1: value 16MHz -> 8MHz; footprint (none) -> Crystal:Crystal_SMD_3225-4Pin_3.2x2.5mm
- renumbered U1 to U2
Connections:
- net +3.3V: now also C2.1, D1.2 (A), J2.1 (Pin_1), J3.1 (Pin_1), J4.1 (Pin_1), R3.1, R4.1, R5.1, U1.2 (VO)
- net GND: now also Y1.2, Y1.4, C1.2, C12.2, C13.2, C2.2, J1.5 (GND), J2.4 (Pin_4), J3.4 (Pin_4), J4.4 (Pin_4), R1.2, U1.1 (GND)
- net HSE_IN: now also Y1.1, C12.1
- net HSE_OUT: now also Y1.3, C13.1
- net SWCLK: now also J3.3 (Pin_3)
- net SWDIO: now also J3.2 (Pin_2)
- net USB_D+: now also J1.3 (D+), R3.2
- net USB_D-: now also J1.2 (D-)
- net I2C2_SCL: now reaches U2.21 (PB10)
- net I2C2_SCL: now also J4.2 (Pin_2), R4.2
- net I2C2_SDA: now reaches U2.22 (PB11)
- net I2C2_SDA: now also J4.3 (Pin_3), R5.2
- net USART1_TX: now reaches U2.42 (PB6)
- net USART1_TX: now also J2.2 (Pin_2)
- net USART1_RX: now reaches U2.43 (PB7)
- net USART1_RX: now also J2.3 (Pin_3)
- new net PWR_LED_K: D1.1 (K), R1.1
- new net VBUS: C1.1, J1.1 (VBUS), U1.3 (VI)
- no-connect marks 0 -> 29
Other:
- note added: "- C3 se coloca en el pin de VDD mas alejado del regulador de 3V3. - Un C de 100n por cada pin de VDD y uno para el pin de VBAT."
- note added: "Calculos segun AN2867: C12, C13 = 2 * (CL - CS) = 2 * (12p - 7p) = 10p C12, C13 = 2 * (CL - CS) = 2 * (12p - 2p) = 20p Se puede adoptar 15p tomando un CS de 5p. - CL se obtiene del Datasheet de Y1. - CS es la capacitancia del PCB más la capacitancia entre los pines PD0 y PD1, y suele valer entre 2p y 7p."
- note added: "El + y - se utilizan para ´poder trazar un par diferencial."
- note added: "Filtrado simetrico para VDDA"
- note added: "LDO 3V3 REGULATOR"
- note added: "MCU STM32F103C8T6"
- note added: "USB / SWD / USART / I2C Connectors"
- note added: "Ver la AN4879 para saber si R3 es necesaria"
- moved on the sheet: C10, C11, C3, C4, C5, C6, C7, C8, C9, FB1, R2, SW1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

Commit message: PCB layout updated
Parts:
- added H1, H2, H3, H4: MountingHole, MountingHole:MountingHole_2.2mm_M2, symbol Mechanical:MountingHole
- SW1: footprint Button_Switch_THT:SW_E-Switch_EG1224_SPDT_Angled -> Button_Switch_SMD:SW_SPDT_PCM12
Other:
- note added: "Mechanical"
- note added: "STM32 Demo Board"
- title: (none) -> STM32 Demo Board
- moved on the sheet: C1, C10, C11, C12, C13, C2, C3, C4, C5, C6, C7, C8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
