File: udemy-learn-kicad-v6-and-stm32-hardware-design.kicad_pcb (KiCad board)
At the start: 4 copper layers, 41 x 31 mm, 32 parts, among them J1 USB_B_Micro, J2 Conn_01x04_Pin, J3 Conn_01x04_Pin, J4 Conn_01x04_Pin, SW1 SW_SPDT, U1 AMS1117-3.3, U2 STM32F103C8T6, Y1 8MHz

Commit message: DFM Completed
Parts:
- moved J4 3.00 mm to (142.4, 88.2)
- moved R1 1.50 mm to (166.0, 82.2)
- moved C10 1.27 mm to (139.2, 80.8)
- moved C9 1.27 mm to (139.2, 79.2)
- moved FB1 1.27 mm to (141.5, 80.0)
- moved R4 1.25 mm to (146.8, 84.0)
- moved R5 1.25 mm to (149.2, 84.0)
- moved R3 0.44 mm to (156.2, 74.4)
- moved C11 0.25 mm to (145.2, 81.2)
- moved C13 0.25 mm to (139.5, 75.0)
- moved C5 0.25 mm to (150.5, 81.2)
Routing:
- net GND: track 0.00 -> 26.9 mm, vias 0 -> 23
- net +3.3V: track 0.00 -> 23.9 mm, vias 0 -> 10
- net /SWDIO: track 0.00 -> 15.6 mm
- net /SWCLK: track 0.00 -> 15.5 mm
- net /USART1_TX: track 0.00 -> 14.7 mm
- net /USART1_RX: track 0.00 -> 14.7 mm
- net /BOOT0: track 0.00 -> 13.8 mm, vias 0 -> 2
- net /USB_D-: track 0.00 -> 13.0 mm
- net /USB_D+: track 0.00 -> 13.0 mm
- net /I2C2_SCL: track 0.00 -> 10.8 mm
- net /I2C2_SDA: track 0.00 -> 10.6 mm
- net /HSE_IN: track 0.00 -> 8.84 mm
- net /NRST: track 0.00 -> 8.80 mm, vias 0 -> 2
- net +3.3VA: track 0.00 -> 7.49 mm
- net /HSE_OUT: track 0.00 -> 6.55 mm
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- added copper zone on F.Cu, net +3.3V
- added copper zone on In2.Cu, net +3.3V
- added copper zone on F.Cu, net GND
- added copper zone on In1.Cu, net GND
- added copper zone on F.Cu, net VBUS
Other:
- outline, holes or cut-outs redrawn
- board text added: "3V3"
- board text added: "BOOT"
- board text added: "GND"
- board text added: "RX"
- board text added: "SCL"
- board text added: "SDA"
- board text added: "SWDIO"
- board text added: "TX"
- board text added: "USB"
- board text added: "V1.0 13/07/2025"
